File: p_bit_ising_machine/p_bit_ising_machine.kicad_sch (KiCad schematic)
At the start: 9 parts

Commit message: Fix all schematic wire gaps and finalize 4-pbit Ising core simulation
Parts:
- removed Cout: 20fF, symbol Device:C
- removed MN_BUF: W=1.5u L=0.18u, symbol eSim_Devices:mosfet_n
- removed MP_BUF: W=3.0u L=0.18u, symbol eSim_Devices:mosfet_p
- removed Rfb: 200k, symbol Device:R
- removed Vin: 0.9V, symbol eSim_Sources:dc
- removed Vnoise: Thermal_Noise, symbol eSim_Sources:pulse
- added C2, C3, C4: 15fF, symbol Device:C
- added Cout1, Cout2, Cout3, Cout4: 20fF, symbol Device:C
- added MN2, MN3, MN4: W=1.0u L=0.18u, symbol eSim_Devices:mosfet_n
- added MN_BUF1, MN_BUF2, MN_BUF3, MN_BUF4: W=1.5u L=0.18u, symbol eSim_Devices:mosfet_n
- added MP2, MP3, MP4: W=2.5u L=0.18u, symbol eSim_Devices:mosfet_p
- added MP_BUF1, MP_BUF2, MP_BUF3, MP_BUF4: W=3.0u L=0.18u, symbol eSim_Devices:mosfet_p
- added Rfb1, Rfb2, Rfb3, Rfb4: 500k, symbol Device:R
- added Vin1, Vin2, Vin3, Vin4: 0.9V, symbol eSim_Sources:dc
- added Vnoise1: Noise_1, symbol eSim_Sources:pulse
- added Vnoise2: Noise_2, symbol eSim_Sources:pulse
- added Vnoise3: Noise_3, symbol eSim_Sources:pulse
- added Vnoise4: Noise_4, symbol eSim_Sources:pulse
Connections:
- net analog_out is gone; now on net GND: C1.1, MN1.1 (D), MP1.3 (S)
- net noise_node is gone; now on net GND: MP1.2 (G)
- net GND: now also C2.1, C2.2, C3.1, C3.2, C4.1, C4.2, Cout1.1, Cout1.2, Cout2.1, Cout2.2, Cout3.1, Cout3.2, Cout4.1, Cout4.2, MN2.1 (D), MN3.1 (D), MN4.1 (D), MN_BUF1.1 (D), MN_BUF2.1 (D), MN_BUF3.1 (D), MN_BUF4.1 (D), MP2.2 (G), MP2.3 (S), MP3.2 (G), MP3.3 (S), MP4.2 (G), MP4.3 (S), MP_BUF1.2 (G), MP_BUF1.3 (S), MP_BUF2.2 (G), MP_BUF2.3 (S), MP_BUF3.2 (G), MP_BUF3.3 (S), MP_BUF4.2 (G), MP_BUF4.3 (S), Rfb1.1, Rfb2.1, Rfb3.1, Rfb4.1
- net VDD: now also MP2.1 (D), MP3.1 (D), MP4.1 (D), MP_BUF1.1 (D), MP_BUF2.1 (D), MP_BUF3.1 (D), MP_BUF4.1 (D)
